File: design/ComplexCalc/ComplexCalc.kicad_pcb (KiCad board)
At the start: 2 copper layers, 111.8 x 112.7 mm, 50 parts, among them J1 V_Battery, J2 Conn_01x09, J3 STLINK, J4 Conn_01x20_Socket, J5 Conn_01x20_Socket, SW1 4, SW10 -, SW11 del, SW12 <-, SW13 7, SW14 8, SW15 9, SW16 M, SW18 MOD, SW19 <, SW2 5, SW20 MOD, SW22 ^, SW23 OK, SW24 v, SW26 MOD, SW27 >, SW28 MOD, SW3 6, SW4 1, SW5 2, SW6 3, SW7 =, SW8 ., SW9 0, U2 AMS1117-3.3, U3 STM32F411CEUx, Y1 8MHz

Commit message: ADC trace connected
Parts:
- moved R8 60.6 mm to (131.6, 28.6), turned to 180 degrees
- moved R7 56.9 mm to (132.3, 24.6)
- moved Y1 9.76 mm to (128.2, 9.25), turned to 0 degrees
- moved D1 8.77 mm to (135.0, 8.05), turned to 180 degrees
- moved U2 8.06 mm to (121.0, 21.0), turned to 90 degrees
- moved C6 6.34 mm to (126.8, 13.8), turned to 0 degrees
- moved C7 5.80 mm to (124.8, 27.1)
- moved R3 5.26 mm to (134.2, 10.9), turned to 90 degrees
- moved C12 4.25 mm to (137.0, 11.2)
- moved R4 3.45 mm to (127.8, 20.8)
- moved C5 3.20 mm to (130.8, 13.7), turned to 180 degrees
- moved R5 3.03 mm to (138.6, 8.10), turned to 0 degrees
- moved C9 2.19 mm to (130.2, 18.9)
- moved C8 1.71 mm to (119.8, 27.4)
- moved J1 1.63 mm to (91.2, 36.1), turned to 180 degrees
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Routing:
- net A0: track 0.00 -> 123.7 mm, vias 0 -> 2
- net 3.3V: track 349.3 -> 379.7 mm
- net GND: track 430.4 -> 444.4 mm
- net C13: track 2.36 -> 6.29 mm
- net Net-(U3-BOOT0): track 3.20 -> 6.64 mm
- net OSC_IN: track 8.05 -> 11.3 mm
- net NRST: track 8.50 -> 10.4 mm
- net OSC_OUT: track 16.1 -> 17.9 mm
- net VIN: track 47.6 -> 48.6 mm
Other:
- board size 111.8 x 112.7 mm -> 97.2 x 112.7 mm
